Commit message: feat: add BrainLab markers config

File: polaris_description/config/polaris.config.xacro (robot description, xacro)
@@ -3,4 +3,5 @@
     <!-- Import polaris ros2_control description -->
     <xacro:include filename="$(find polaris_description)/ros2_control/polaris.ros2_control.xacro" />
+		<link name="polaris_frame"/>
     <xacro:ndi_sensor name="polaris"/>
 </robot>

File: polaris_description/ros2_control/polaris.ros2_control.xacro (robot description, xacro)
@@ -6,11 +6,9 @@
       <hardware>
         <plugin>ndi_hardware/NdiSensorHardwareInterface</plugin>
-        <param name="ndi_ip">192.155.1.80</param>
+        <param name="ndi_ip">169.254.1.10</param>
       </hardware>
       <!-- repeat this part for multiple trackers -->
-      <xacro:tracker name="fus_tracker"
-        srom="/home/adnan/Desktop/ros2/ndisys_ros2/polaris_description/srom/UfoGuideTransducer.rom" />
-      <xacro:tracker name="needle"
-        srom="/home/adnan/Desktop/ros2/ndisys_ros2/polaris_description/srom/8700340.rom" />
+      <xacro:tracker name="brainlab_reference1"
+        srom="$(find polaris_description)/srom/BrainLabReference1.rom" />
     </ros2_control>
   </xacro:macro>
